File: pcb/hex-board/hex-board.kicad_pcb (KiCad board)
At the start: 2 copper layers, 77.1 x 89 mm, 21 parts

Commit message: Added JST connector to hex board
Parts:
- removed +5V, GND: TestPoint_Pad_2.0x2.0mm, TestPoint:TestPoint_Pad_2.0x2.0mm
- removed DATA IN: TestPoint_Pad_2.0x2.0mm, TestPoint:TestPoint_Pad_2.0x2.0mm
- added J1: Conn_01x04_Socket, Connector_JST:JST_EH_S4B-EH_1x04_P2.50mm_Horizontal, B.Cu at (159.6, 79.9)
Routing:
- net Data IN: track 3.94 -> 13.0 mm, vias 1 -> 0
- net GND: track 32.2 -> 38.6 mm, vias 19 -> 18
- net +5V: track 487.5 -> 491.2 mm, vias 14 -> 13
